File: Nafanya_Keyboard/Nafanya_Keyboard.kicad_pcb (KiCad board)
At the start: 2 copper layers, 200 x 91 mm, 55 parts, among them J1 KEYBOARD_TO_NAFANYA, SW1 1, SW10 T, SW11 A, SW12 S, SW13 D, SW14 F, SW15 G, SW16 CAPS_SHIFT, SW17 Z, SW18 X, SW19 C, SW2 2, SW20 V, SW21 6, SW22 Y, SW23 H, SW24 B, SW25 7, SW26 U, SW27 J, SW28 N, SW29 8, SW3 3, SW30 I, SW31 K, SW32 M, SW33 9, SW34 O, SW35 L, SW36 SYMBOL_SHIFT, SW37 0, SW38 P, SW39 ENTER, SW4 4, SW40 BREAK_SPACE, SW41 RESET, SW5 5, SW6 Q, SW7 W, SW8 E, SW9 R

Commit message: Initial keyboard PCB designed
Parts:
- removed H9: Speaker, MountingHole:MountingHole_3.2mm_M3
- added J2: Columns, Connector_PinHeader_2.54mm:PinHeader_1x05_P2.54mm_Horizontal, B.Cu at (172.5, 66.0)
- added J3: Rows, Connector_PinHeader_2.54mm:PinHeader_1x08_P2.54mm_Horizontal, B.Cu at (133.8, 66.0)
- added J4: Faceplate GND, Connector_PinSocket_2.54mm:PinSocket_1x01_P2.54mm_Vertical, B.Cu at (78.0, 142.0)
- H1, H8, LS1: moved to B.Cu
- J1: value KEYBOARD_TO_NAFANYA -> Speaker/Reset/Power; footprint Connector_PinHeader_2.54mm:PinHeader_1x17_P2.54mm_Horizontal -> Connector_PinHeader_2.54mm:PinHeader_1x04_P2.54mm_Horizontal; moved to B.Cu
- SW10: value T -> 0
- SW11: value A -> Q
- SW12: value S -> W
- SW13: value D -> E
- SW14: value F -> R
- SW15: value G -> T
- SW16: value CAPS_SHIFT -> Y
- SW17: value Z -> U
- SW18: value X -> I
- SW19: value C -> O
- SW20: value V -> P
- SW21: value 6 -> A
- SW22: value Y -> S
- SW23: value H -> D
- SW24: value B -> F
- SW25: value 7 -> G
- SW26: value U -> H
- SW28: value N -> K
- SW29: value 8 -> L
- SW30: value I -> ENTER
- SW31: value K -> CAPS_SHIFT
- SW32: value M -> Z
- SW33: value 9 -> X
- SW34: value O -> C
- SW35: value L -> V
- SW36: value SYMBOL_SHIFT -> B
- SW37: value 0 -> N
- SW38: value P -> M
- SW39: value ENTER -> SYMBOL_SHIFT
- SW6: value Q -> 6
- SW7: value W -> 7
- SW8: value E -> 8
- SW9: value R -> 9
- moved SW31 165.1 mm to (67.0, 128.8)
- moved SW22 152.8 mm to (84.0, 114.8)
- moved SW36 150.7 mm to (152.0, 128.8)
- moved SW32 148.4 mm to (83.7, 128.8)
- moved SW37 140.3 mm to (169.0, 128.8)
- moved SW29 139.3 mm to (202.8, 114.8)
- moved SW23 137.6 mm to (100.9, 114.8)
- moved SW30 136.7 mm to (219.8, 114.8)
- moved SW33 132.0 mm to (101.0, 128.8)
- moved SW38 131.7 mm to (186.0, 128.8)
- moved SW39 125.5 mm to (203.0, 128.8)
- moved SW24 123.6 mm to (117.9, 114.8)
- moved SW10 123.1 mm to (219.8, 86.8)
- moved SW9 122.7 mm to (206.0, 89.0)
- moved SW40 122.0 mm to (220.0, 128.8)
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Connections:
- J1 pad 1: GND -> SPEAKER
- J1 pad 2: ROW6 -> GND
- J1 pad 4: ROW7 -> +5V
- SW10 pad 1: COL5 -> COL1
- SW10 pad 2: ROW2 -> ROW5
- SW11 pad 2: ROW3 -> ROW2
- SW12 pad 2: ROW3 -> ROW2
- SW13 pad 2: ROW3 -> ROW2
- SW14 pad 2: ROW3 -> ROW2
- SW15 pad 2: ROW3 -> ROW2
- SW16 pad 1: COL1 -> COL5
- SW16 pad 2: ROW4 -> ROW6
- SW17 pad 1: COL2 -> COL4
- SW17 pad 2: ROW4 -> ROW6
- SW18 pad 2: ROW4 -> ROW6
- SW19 pad 1: COL4 -> COL2
- SW19 pad 2: ROW4 -> ROW6
- SW20 pad 1: COL5 -> COL1
- SW20 pad 2: ROW4 -> ROW6
- SW21 pad 1: COL5 -> COL1
- SW21 pad 2: ROW5 -> ROW3
- SW22 pad 1: COL5 -> COL2
- SW22 pad 2: ROW6 -> ROW3
- SW23 pad 1: COL5 -> COL3
- SW23 pad 2: ROW7 -> ROW3
- SW24 pad 1: COL5 -> COL4
- SW24 pad 2: ROW8 -> ROW3
- SW25 pad 1: COL4 -> COL5
- SW25 pad 2: ROW5 -> ROW3
- SW26 pad 1: COL4 -> COL5
- SW26 pad 2: ROW6 -> ROW7
- SW28 pad 1: COL4 -> COL3
- SW28 pad 2: ROW8 -> ROW7
- SW29 pad 1: COL3 -> COL2
- SW29 pad 2: ROW5 -> ROW7
- SW30 pad 1: COL3 -> COL1
- SW30 pad 2: ROW6 -> ROW7
- SW31 pad 1: COL3 -> COL1
- SW31 pad 2: ROW7 -> ROW4
- SW32 pad 1: COL3 -> COL2
- SW32 pad 2: ROW8 -> ROW4
- SW33 pad 1: COL2 -> COL3
- SW33 pad 2: ROW5 -> ROW4
- SW34 pad 1: COL2 -> COL4
- SW34 pad 2: ROW6 -> ROW4
- SW35 pad 1: COL2 -> COL5
- SW35 pad 2: ROW7 -> ROW4
- SW36 pad 1: COL2 -> COL5
- SW37 pad 1: COL1 -> COL4
- SW37 pad 2: ROW5 -> ROW8
- SW38 pad 1: COL1 -> COL3
- SW38 pad 2: ROW6 -> ROW8
- SW39 pad 1: COL1 -> COL2
- SW39 pad 2: ROW7 -> ROW8
- SW6 pad 1: COL1 -> COL5
- SW6 pad 2: ROW2 -> ROW5
- SW7 pad 1: COL2 -> COL4
- SW7 pad 2: ROW2 -> ROW5
- SW8 pad 2: ROW2 -> ROW5
- SW9 pad 1: COL4 -> COL2
- SW9 pad 2: ROW2 -> ROW5
Routing:
- net COL1: track 0.00 -> 307.5 mm
- net COL2: track 0.00 -> 278.8 mm, vias 0 -> 1
- net COL3: track 0.00 -> 251.3 mm
- net COL4: track 0.00 -> 213.1 mm
- net COL5: track 0.00 -> 180.7 mm, vias 0 -> 1
- net ROW8: track 0.00 -> 180.2 mm
- net ROW3: track 0.00 -> 173.6 mm
- net ROW4: track 0.00 -> 168.7 mm
- net ROW7: track 0.00 -> 166.0 mm
- net ROW6: track 0.00 -> 150.2 mm
- net ROW2: track 0.00 -> 145.2 mm
- net ROW5: track 0.00 -> 141.0 mm
- net RESET: track 0.00 -> 140.7 mm
- net SPEAKER: track 0.00 -> 131.7 mm
- net ROW1: track 0.00 -> 117.8 mm
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- added copper zone on B.Cu, net GND
Other:
- board size 200 x 91 mm -> 190 x 101 mm
- board text added: "5 4 3 2 1"
- board text added: "8 7 6 5 4 3 2 1"
- board text added: "Brett Hallen, Apr 2025 Port Macquarie, Australia www.youtube.com/@Brfff"
- board text added: "Speaker GND Reset +5V"
- board text added: "НАФАНЯ"

Commit message: Refining PCB layout
Parts:
- moved SW10 8.00 mm to (211.8, 86.8)
- moved SW19 8.00 mm to (194.5, 100.8)
- moved SW20 8.00 mm to (211.5, 100.8)
- moved SW29 8.00 mm to (194.8, 114.8)
- moved SW30 8.00 mm to (211.8, 114.8)
- moved SW39 8.00 mm to (195.0, 128.8)
- moved SW40 8.00 mm to (212.0, 128.8)
- moved SW41 8.00 mm to (194.8, 71.8)
- moved SW9 8.00 mm to (198.0, 89.0)
- moved H6 7.00 mm to (143.0, 148.0)
- moved H7 7.00 mm to (143.0, 56.0)
- moved SW17 7.00 mm to (161.6, 100.8)
- moved SW18 7.00 mm to (178.6, 100.8)
- moved SW27 7.00 mm to (161.8, 114.8)
- moved SW28 7.00 mm to (178.8, 114.8)
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Routing:
- net ROW6: track 150.2 -> 161.2 mm, vias 0 -> 1
- net ROW5: track 141.0 -> 130.4 mm, vias 0 -> 1
- net COL3: track 251.3 -> 242.3 mm
- net RESET: track 140.7 -> 132.7 mm
- net COL5: track 180.7 -> 187.8 mm
- net COL4: track 213.1 -> 219.2 mm
- net COL2: track 278.8 -> 284.3 mm, vias 1 -> 0
- net ROW8: track 180.2 -> 175.3 mm
- net ROW7: track 166.0 -> 161.5 mm
- net ROW4: track 168.7 -> 166.1 mm
- net ROW1: track 117.8 -> 115.5 mm
- net COL1: track 307.5 -> 305.2 mm, vias 0 -> 1
- net ROW2: track 145.2 -> 144.5 mm
- net ROW3: track 173.6 -> 174.2 mm
Other:
- board size 190 x 101 mm -> 192 x 101 mm
- board text added: "Col 1"
- board text added: "Col 2"
- board text added: "Col 3"
- board text added: "Col 4"
- board text added: "Col 5"
- board text added: "Row 1"
- board text added: "Row 2"
- board text added: "Row 3"
- board text added: "Row 4"
- board text added: "Row 5"
- board text added: "Row 6"
- board text added: "Row 7"
- board text added: "Row 8"

Commit message: Finalised layout
Parts:
- removed RN1: 9.1KΩ, Resistor_THT:R_Array_SIP9
- added R2: 10KΩ, Resistor_THT:R_Axial_DIN0207_L6.3mm_D2.5mm_P7.62mm_Horizontal, F.Cu at (95.3, 79.0)
- added R3: 10KΩ, Resistor_THT:R_Axial_DIN0207_L6.3mm_D2.5mm_P7.62mm_Horizontal, F.Cu at (99.3, 79.0)
- added R4: 10KΩ, Resistor_THT:R_Axial_DIN0207_L6.3mm_D2.5mm_P7.62mm_Horizontal, F.Cu at (103.3, 79.0)
- added R5: 10KΩ, Resistor_THT:R_Axial_DIN0207_L6.3mm_D2.5mm_P7.62mm_Horizontal, F.Cu at (107.3, 79.0)
- added R6: 10KΩ, Resistor_THT:R_Axial_DIN0207_L6.3mm_D2.5mm_P7.62mm_Horizontal, F.Cu at (111.3, 79.0)
- added R7: 10KΩ, Resistor_THT:R_Axial_DIN0207_L6.3mm_D2.5mm_P7.62mm_Horizontal, F.Cu at (115.3, 79.0)
- added R8: 10KΩ, Resistor_THT:R_Axial_DIN0207_L6.3mm_D2.5mm_P7.62mm_Horizontal, F.Cu at (119.3, 79.0)
- added R9: 10KΩ, Resistor_THT:R_Axial_DIN0207_L6.3mm_D2.5mm_P7.62mm_Horizontal, F.Cu at (123.3, 79.0)
- SW41: value RESET -> RESET/СБРОС
- moved J1 112.3 mm to (179.2, 60.5)
- moved J2 12.6 mm to (159.9, 66.6)
- moved R1 7.62 mm to (91.3, 71.4), turned to -90 degrees
- moved SW30 4.81 mm to (216.0, 117.0)
- moved SW29 4.78 mm to (199.0, 117.0)
- moved SW27 4.74 mm to (166.0, 117.0)
- moved SW20 4.67 mm to (216.0, 102.0)
- moved SW19 4.64 mm to (199.0, 102.0)
- moved SW23 4.64 mm to (99.0, 117.0)
- moved SW17 4.59 mm to (166.0, 102.0)
- moved SW33 4.59 mm to (99.0, 131.0)
- moved SW37 4.59 mm to (166.0, 131.0)
- moved SW39 4.59 mm to (199.0, 131.0)
- moved SW40 4.59 mm to (216.0, 131.0)
- moved SW13 4.48 mm to (99.0, 102.0)
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Connections:
- J1 pad 1: SPEAKER -> +5V
- J1 pad 4: +5V -> SPEAKER
Routing:
- net SPEAKER: track 131.7 -> 9.37 mm
- net RESET: track 132.7 -> 22.4 mm
- net +5V: track 29.9 -> 96.1 mm
- net ROW6: track 161.2 -> 145.2 mm, vias 1 -> 0
- net ROW3: track 174.2 -> 160.5 mm
- net COL5: track 187.8 -> 176.1 mm
- net COL3: track 242.3 -> 253.0 mm
- net COL2: track 284.3 -> 274.1 mm, vias 0 -> 1
- net COL4: track 219.2 -> 210.8 mm
- net ROW4: track 166.1 -> 173.8 mm
- net ROW8: track 175.3 -> 171.9 mm
- net COL1: track 305.2 -> 308.2 mm
- net ROW1: track 115.5 -> 117.7 mm
- net ROW5: track 130.4 -> 132.7 mm, vias 1 -> 0
- net ROW7: track 161.5 -> 159.3 mm
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Other:
- board size 192 x 101 mm -> 193 x 102.2 mm
- board text added: "10мм"
- board text added: "14мм"
- board text added: "17мм"
- board text added: "Принтер Тест"
